File: T41Expander.kicad_pcb (KiCad board)
At the start: 2 copper layers, 83.6 x 79.8 mm, 104 parts, among them J1 Conn_XT30, J10 Conn_01x04, J11 Conn_01x04, J12 Conn_01x02, J13 Conn_01x02, J14 Conn_01x02, J15 Conn_01x04, J16 Conn_01x03, J17 Conn_01x03, J18 Conn_01x03, J19 Conn_01x03, J2 Conn_01x04, J20 Conn_01x03, J21 Conn_01x03, J22 Conn_01x04, J23 Conn_01x04, J24 Conn_01x04, J25 Conn_01x04, J26 Conn_01x04, J3 Conn_01x04, J4 Conn_XT30F, J5 Conn_01x04, J6 Conn_01x04, J7 Conn_XT30F, J8 Conn_01x04, J9 Conn_01x04, Q1 BTS117, Q2 BTS117, U1 MIC29502WT, U2 TSR_2-2450, U3 Teensy4.1

Commit message: T41Expander V1.0 envoyé en fabrication
Other:
- board text added: "Servos"
- board text added: "TEENSY 4.1"
Changed lines of the file:
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@@
   (general
     (thickness 1.6)
-    (drawings 48)
+    (drawings 50)
     (tracks 583)
     (zones 0)
@@
       (drillshape 0)
       (scaleselection 1)
-      (outputdirectory "export"))
+      (outputdirectory "./gerber"))
   )
   (net 0 "")
@@
     (tags resistor)
     (attr smd)
-    (fp_text reference R28 (at -3.05608 0.0508 90) (layer B.SilkS)
+    (fp_text reference R28 (at -0.0538 1.83896 180) (layer B.SilkS)
       (effects (font (size 0.8 0.8) (thickness 0.15)) (justify mirror))
     )
@@
     )
   )
+  (gr_text "TEENSY 4.1" (at 61.595 53.82768) (layer F.SilkS)
+    (effects (font (size 1 1) (thickness 0.15)))
+  )
+  (gr_text Servos (at 46.57344 29.33192) (layer F.SilkS)
+    (effects (font (size 1 1) (thickness 0.15)))
+  )
   (gr_text VBAT (at 34.59988 35.13328) (layer B.SilkS)
     (effects (font (size 1 1) (thickness 0.15)) (justify mirror))
   )
-  (gr_text + (at 95.03156 25.47112) (layer F.SilkS)
+  (gr_text - (at 95.03156 25.47112) (layer F.SilkS)
     (effects (font (size 1 1) (thickness 0.15)))
   )
